File: vcu/Power.kicad_sch (KiCad schematic)
At the start: 36 parts, among them IC1 MAX20040DATPA_VY+, J11 PWR, U11 LMR33630CDDA, U12 LD1117S33TR_SOT223

Commit message: added planned change notes
mwuhahahahahhah im tearing this thing to pieces
Other:
- note added: "Planned changes: - add zenner+fet reverse protection - decide if using a powerplexer for 5v in opt - unify grounds - remove option to power sensors from vcu - rename power nets - add 12v -> 5v buck - add 5v -> 3.3v ldo OR - add 12V -> 3.3v ldo/buck - add fuckass inductor Because: - stop people frying board - vcu is a single point failure, any excess power stuff like the sensor supply should be se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"
Changed lines of the file:
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@@
+		)
+	)
+	(text "Planned changes:\n- add zenner+fet reverse protection \n- decide if using a powerplexer for 5v in opt\n- unify grounds\n- remove option to power sensors from vcu\n- rename power nets \n- add 12v -> 5v buck\n- add 5v -> 3.3v ldo\nOR\n- add 12V -> 3.3v ldo/buck\n- add fuckass inductor\n\nBecause:\n- stop people frying board\n- vcu is a single point failure, any excess power\n  stuff like the sensor supply should be seperated\n- sensors should instead be powered from a REGULATED,\n  CONTINUOUS supply, ie a Sensor Power Module in the dash\n- +12V is NOT 12V AS IT IS STRAIGHT OFF THE BATTERY AND \n  NOT REGULATED!!! Will rename nets to convey this"
+		(exclude_from_sim no)
+		(at 150.114 111.252 0)
+		(effects
+			(font
+				(size 1.27 1.27)
+				(color 255 153 0 1)
+			)
+			(justify left)
 		)
 	)
