File: vcu/input-shift.kicad_sch (KiCad schematic)
At the start: 45 parts, among them U3 TLV274, U4 HCF4010, U5 ILQ615-4X009T

Commit message: added planned change notes
mwuhahahahahhah im tearing this thing to pieces
Other:
- note added: "Planned changes: - check if optoiso is the best choice - swap for a much smaller package - double number of inputs Why: - future proofing - space will be an issue on this board, so trying to keep things neat"
- note added: "Planned changes: - double number of channels - proper input clamping - use 2.5vref - make input voltage configurable via jumpers - add spice sims - add more filter stages - unify grounds Because: - make readings nicer (anti-aliasing) - protect from transience - any sensor can be connected up to each channel so more cusomisable"
Changed lines of the file:
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@@
+		)
+	)
+	(text "Planned changes:\n- check if optoiso is the best choice\n- swap for a much smaller package\n- double number of inputs\n\nWhy:\n- future proofing\n- space will be an issue on this board, so \n  trying to keep things neat\n"
+		(exclude_from_sim no)
+		(at 256.032 111.252 0)
+		(effects
+			(font
+				(size 1.27 1.27)
+				(color 255 153 0 1)
+			)
+			(justify left)
 		)
 	)
@@
 		)
 	)
+	(text "Planned changes:\n- double number of channels\n- proper input clamping\n- use 2.5vref\n- make input voltage configurable via jumpers\n- add spice sims\n- add more filter stages\n- unify grounds\n\nBecause:\n- make readings nicer (anti-aliasing)\n- protect from transience\n- any sensor can be connected up to each channel\n  so more cusomisable"
+		(exclude_from_sim no)
+		(at 166.624 51.816 0)
+		(effects
+			(font
+				(size 1.27 1.27)
+				(color 255 153 0 1)
+			)
+			(justify left)
+		)
+	)
