File: vcu/mcu.kicad_sch (KiCad schematic)
At the start: 63 parts, among them IC3 HT16K33, J10 Conn_ARM_JTAG_SWD_20, J9 USB_C_Receptacle_USB2.0_16P, SW1 SW_Push, SW2 SW_SPDT, U6 STM32F746ZGT6, Y1 8MHz

Commit message: added planned change notes
mwuhahahahahhah im tearing this thing to pieces
Other:
- note added: "Because: - Remove excess debug for space - Not needed during running - Using expansion slots debug can be accessed when needed - Faster clock, CANFD, IMU for future proofing - EEPROM for config flashing - Boot pad for space - Keeping jtag cuz goated - SD card for logging - temp sensor so board can have thermal shutoff/reg the h7/f7 do have internal ones but they r shit"
- note added: "Planned changes: - higher clock - smaller JTAG header (6 pin micro) - remove 7 seg - remove uart - change to CANFD/-+58V fault compat can trancivers - add transient protection to can trancivers - add rs232/3rd can - add sd card - fix grounding - add pads for boot - smaller rst button - faster clock - add temp sensor - add imu? - add eeprom - add header for expansion slot with periherals and GPIO"
Changed lines of the file:
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@@
+		)
+	)
+	(text "Planned changes:\n- higher clock\n- smaller JTAG header (6 pin micro)\n- remove 7 seg\n- remove uart\n- change to CANFD/-+58V fault compat can trancivers\n- add transient protection to can trancivers\n- add rs232/3rd can \n- add sd card\n- fix grounding\n- add pads for boot\n- smaller rst button\n- faster clock\n- add temp sensor\n- add imu?\n- add eeprom\n- add header for expansion slot with\n  periherals and GPIO"
+		(exclude_from_sim no)
+		(at 185.928 74.422 0)
+		(effects
+			(font
+				(size 1.27 1.27)
+				(color 255 153 0 1)
+			)
+			(justify left)
 		)
 	)
@@
 		)
 	)
+	(text "Because:\n- Remove excess debug for space\n- Not needed during running\n- Using expansion slots debug can be accessed\n  when needed\n- Faster clock, CANFD, IMU for future proofing\n- EEPROM for config flashing\n- Boot pad for space\n- Keeping jtag cuz goated\n- SD card for logging\n- temp sensor so board can have thermal shutoff/reg\n  the h7/f7 do have internal ones but they r shit"
+		(exclude_from_sim no)
+		(at 230.886 90.17 0)
+		(effects
+			(font
+				(size 1.27 1.27)
+				(color 255 153 0 1)
+			)
+			(justify left)
+		)
+	)
