File: vcu/output-shift.kicad_sch (KiCad schematic)
At the start: 11 parts, among them U10 HCF4010, U9 ILQ615-4X009T

Commit message: added planned change notes
mwuhahahahahhah im tearing this thing to pieces
Other:
- note added: "Planned changes: - double output channels and intergrate with fet array on main - decide if to use fets or optoisos - could have all the same or low speed and high speed options - might add 5v input capabilities Because: - channels can be multipurpose - space saving - switching speed"
Changed lines of the file:
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@@
+		)
+	)
+	(text "Planned changes:\n- double output channels and intergrate with fet array on main\n- decide if to use fets or optoisos\n- could have all the same or low speed and high speed options\n- might add 5v input capabilities\n\nBecause:\n- channels can be multipurpose\n- space saving\n- switching speed"
+		(exclude_from_sim no)
+		(at 24.13 101.854 0)
+		(effects
+			(font
+				(size 1.27 1.27)
+				(color 255 153 0 1)
+			)
+			(justify left)
 		)
 	)
