File: vcu/vcu.kicad_pcb (KiCad board)
At the start: 4 copper layers, 157 parts, among them IC1 MAX20040DATPA_VY+, J10 Conn_ARM_JTAG_SWD_20, J11 PWR, J6 FSUK_RTD, J8 OUT, Q1 FDN359BN, Q2 FDN359BN, Q3 FDN359BN, Q4 FDN359BN, Q5 FDN359BN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

Commit message: added planned change notes
mwuhahahahahhah im tearing this thing to pieces
Parts:
- moved U6 2.93 mm to (223.1, 119.5)
Changed lines of the file:
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@@
 	(footprint "Package_QFP:LQFP-144_20x20mm_P0.5mm"
 		(layer "F.Cu")
-		(at 223.139 122.428)
+		(at 223.139 119.5)
 		(descr "LQFP, 144 Pin (http://ww1.microchip.com/downloads/en/PackagingSpec/00000049BQ.pdf#page=425), generated with kicad-footprint-generator ipc_gullwing_generator.py")
 		(tags "LQFP QFP")
