File: vcu/vcu.kicad_sch (KiCad schematic)
At the start: 43 parts, among them J1 Front Logic IO, J12 Analogue Power, J2 Analogue Inputs, J5 Spare GPIO, J6 FSUK_RTD, J7 CAN, J8 Rear Logic IO, Q1 FDN359BN, Q2 FDN359BN, Q3 FDN359BN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

Commit message: added planned change notes
mwuhahahahahhah im tearing this thing to pieces
Other:
- note added: "Planned changes: - add test points - fix analog setup - remove analog supply - redo schematic formatting to improve readability - unify connectors - add expansion header for modularity Because: - better protect board from transience - make loom making easier - future proof board - splitting grounds is extremely difficult to do and not nessacary in this use case - test points to assist debug"
Changed lines of the file:
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@@
+		)
+	)
+	(text "Planned changes:\n- add test points\n- fix analog setup\n- remove analog supply\n- redo schematic formatting to improve\n  readability\n- unify connectors\n- add expansion header for modularity\n\nBecause:\n- better protect board from transience\n- make loom making easier\n- future proof board\n- splitting grounds is extremely difficult to do\n  and not nessacary in this use case\n- test points to assist debug\n"
+		(exclude_from_sim no)
+		(at 156.464 46.482 0)
+		(effects
+			(font
+				(size 1.27 1.27)
+				(color 255 153 0 1)
+			)
+			(justify left)
 		)
 	)
