File: CANna-VCU/CANna-VCU.kicad_sch (KiCad schematic)
At the start: 0 parts

Commit message: first draft of full board
Parts:
- added H1, H2, H3, H4: M3, MountingHole:MountingHole_3.2mm_M3, symbol Mechanical:MountingHole
Other:
- sheet Protected IO renamed HSIO
- added sheet LSIO (vcu_lsio.kicad_sch)
- note added: "Mounting Holes"
