File: CANna-VCU/vcu_mcu.kicad_sch (KiCad schematic)
At the start: 3 parts, among them J9 USB_C_Receptacle_USB2.0_16P, U3 M24256-DRD, U6 STM32F746ZGT6

Commit message: first draft of full board
Parts:
- added C1: 0.1uF, Capacitor_SMD:C_0402_1005Metric, symbol Device:C
- added C10: 4.7uF, Capacitor_SMD:C_0402_1005Metric, symbol Device:C
- added C11, C12, C13, C17, C18, C4, C9: 100nF, Capacitor_SMD:C_0402_1005Metric, symbol Device:C
- added C14, C16: 2.2u, Capacitor_SMD:C_0805_2012Metric_Pad1.18x1.45mm_HandSolder, symbol Device:C
- added C15: 100nF, Capacitor_SMD:C_0603_1608Metric, symbol Device:C
- added C19: 1uF, Capacitor_SMD:C_0402_1005Metric, symbol Device:C
- added C2: 10uF, Capacitor_SMD:C_0402_1005Metric, symbol Device:C
- added C3: 68nF, Capacitor_SMD:C_0402_1005Metric, symbol Device:C
- added C5, C6: 100n, Capacitor_SMD:C_0402_1005Metric, symbol Device:C
- added C7, C8: 4.7pF, Capacitor_SMD:C_0402_1005Metric, symbol Device:C
- added J1: Conn_02x20_Odd_Even, symbol Connector_Generic:Conn_02x20_Odd_Even
- added J3: SD_Card_Device, Connector_Card:SD_Hirose_DM1AA_SF_PEJ82, symbol Connector:SD_Card_Device
- added J4: CLP-103-02-F-D, symbol Connector:Conn_01x06_Socket
- added R1, R2: 5.1k, Resistor_SMD:R_0402_1005Metric, symbol Device:R
- added R3: 100K, Resistor_SMD:R_0402_1005Metric, symbol Device:R
- added R4: 1.3K, Resistor_SMD:R_0402_1005Metric, symbol Device:R
- added R5, R6: 10K, Resistor_SMD:R_0402_1005Metric, symbol Device:R
- added R7, R8: 2.2K, Resistor_SMD:R_0402_1005Metric, symbol Device:R
- added SW1, SW2: CK_KMS2xxG, Button_Switch_SMD:SW_SPST_CK_KMS2xxGP, symbol Switch:CK_KMS2xxG
- added U2: MCP9800Ax-xOT, Package_TO_SOT_SMD:SOT-23-5, symbol Sensor_Temperature:MCP9800Ax-xOT
- added U3: ISM330DHCX, Package_LGA:LGA-14_3x2.5mm_P0.5mm_LayoutBorder3x4y, symbol Sensor_Motion:ISM330DHCX
- added Y1: 25MHz, Crystal:Crystal_SMD_3225-4Pin_3.2x2.5mm_HandSoldering, symbol Device:Crystal_GND24
- renumbered J9 to J2, U3 to U1, U6 to U4
Connections:
- net GND: now reaches J2.A1 (GND), J2.A12 (GND), J2.B1 (GND), J2.B12 (GND)
- net GND: now also J2.S1 (SHIELD), U1.4 (VSS), U4.107 (VSS), U4.120 (VSS), U4.130 (VSS), U4.16 (VSS), U4.31 (VSSA), U4.38 (VSS), U4.51 (VSS), U4.61 (VSS), U4.83 (VSS), U4.94 (VSS), C1.1, C10.2, C11.2, C12.2, C13.2, C14.1, C15.2, C16.1, C17.2, C18.2, C19.2, C2.1, C3.1, C4.1, C5.1, C6.1, C7.2, C8.2, C9.2, J3.3 (VSS), J3.6 (VSS), J4.6 (Pin_6), R1.1, R2.1, SW1.2, SW1.SH (B), SW2.2, SW2.SH (B), U2.2 (GND), U3.2 (SDx), U3.3 (SCx), U3.6 (GND), U3.7 (GND), Y1.2, Y1.4
- net +5V_UNPROT: now reaches J2.A4 (VBUS), J2.A9 (VBUS), J2.B4 (VBUS), J2.B9 (VBUS)
- net at J2.A5 (CC1): now also R1.2
- net USB_D+: now reaches J2.A6 (D+)
- net USB_D+: now also J2.B6 (D+), U4.104 (PA12)
- net USB_D-: now reaches J2.A7 (D-)
- net USB_D-: now also J2.B7 (D-), U4.103 (PA11)
- net at J2.B5 (CC2): now also R2.2
- net +3V3: now reaches U1.1 (E0)
- net +3V3: now also U1.2 (E1), U1.3 (E2), U1.8 (VCC), U4.108 (VDD), U4.121 (VDD), U4.131 (VDD), U4.144 (VDD), U4.17 (VDD), U4.30 (VDD), U4.39 (VDD), U4.52 (VDD), U4.6 (VBAT), U4.62 (VDD), U4.72 (VDD), U4.84 (VDD), U4.95 (VDDUSB), C1.2, C10.1, C11.1, C12.1, C13.1, C15.1, C17.1, C2.2, C4.2, C5.2, C6.2, C9.1, J3.4 (VDD), J4.5 (Pin_5), R3.2, R5.2, R6.2, R7.2, R8.2, SW1.1, SW2.1, U2.1 (V_{DD}), U3.5 (VDDIO), U3.8 (VDD)
- net I2C_SDA: now reaches U1.5 (SDA)
- net I2C_SDA: now also U4.140 (PB9), R7.1, U2.5 (SDA), U3.14 (SDA)
- net I2C_SCL: now reaches U1.6 (SCL)
- net I2C_SCL: now also U4.139 (PB8), R8.1
- net EEPROM_WC: now reaches U1.7 (WC)
- net UART_CLK: now reaches U4.100 (PA8)
- net UART_TX: now reaches U4.101 (PA9)
- net UART_RX: now reaches U4.102 (PA10)
- net SWDIO: now reaches U4.105 (PA13)
- net SWDIO: now also J4.4 (Pin_4)
- net at U4.106 (VCAP_2): now also C16.2
- net SWCLK: now reaches U4.109 (PA14)
- net SWCLK: now also J4.3 (Pin_3)
- net CAN0_RX: now reaches U4.114 (PD0)
- net CAN0_TX: now reaches U4.115 (PD1)
- net SWO: now reaches U4.133 (PB3)
- net SWO: now also J4.1 (Pin_1)
- net nRST: now reaches U4.134 (PB4)
- net nRST: now also C3.2, J4.2 (Pin_2), R3.1
- net CAN1_TX: now reaches U4.136 (PB6)
- net BOOT_0: now reaches U4.138 (BOOT0)
- net OSC_IN: now reaches U4.23 (PH0)
- net OSC_IN: now also C8.1, Y1.1
- net OSC_OUT: now reaches U4.24 (PH1)
- net OSC_OUT: now also R4.1
- net RST: now reaches U4.25 (NRST)
- net RST: now also R5.1
- net +3V3A: now reaches U4.33 (VDDA)
- net +3V3A: now also C18.1, C19.1
- net at U4.71 (VCAP_1): now also C14.2
- net CAN1_RX: now reaches U4.73 (PB12)
- new net: C7.1, R4.2, Y1.3
- new net BOOT: R6.1
- new net I2C_CLK: U2.4 (SCLK), U3.13 (SCL)
- new net IMU_ADDR: U3.1 (SDO/SA0)
- new net IMU_INTR1: U3.4 (INT1)
- new net IMU_INTR2: U3.9 (INT2)
- new net IMU_MODE: U3.12 (CS)
- new net SPI_CLK: J3.5 (CLK)
- new net SPI_CS_SD: J3.1 (CD/DAT3)
- new net SPI_MISO: J3.7 (DAT0)
- new net SPI_MOSI: J3.2 (CMD)
- new net TOO_HOT: U2.3 (ALERT)
- no-connect marks 0 -> 6
Other:
- note added: "**ADD REVERSE PROT IN PWR SHEET**"
- note added: "**CHECK CAP VALUE AND PULLUP**"
- note added: "**CHECK DEBOUNCE** **CHECK IO DIRECTIONS**"
- note added: "**CHECK FOOTPRINT** **CHECK IO DIRECTION**"
- note added: "**CHECK I2C ADDR**"
- note added: "**CHOOSE CONNECTOR**"
- note added: "**PULLUPS???**"
- note added: "**SPEC CAP**"
- note added: "**WATCH IDs**"
- note added: "**WATCH SD POWER**"
- note added: "- ALERT pulls @ configurable temp - place this guy in sensor in dense area - added temp so we have an idea how hot the vcu box gets - could be used to thermal shutdown"
- note added: "- UMU_INTR1/2 are programmable interrupts - IMU_MODE decides operation mode of chip - check if any extra bulk caps needed - this is footprint compatible with other st IMUs - this one has some ai bs idk - up to rob which one we use"
- note added: "- bulk capacitence needed = 10pF - assume parasitic of 7pf CL1/L2 = 10 - 7 * 2 = 6pF - closest standard value = 4.7 - nice caps should be chosen, ideally np0/c0g"
- note added: "- is eeprom acc needed??? - cant u just flash to the f7 eeprom? - stuck with previously specced one - has 256kb flash as 32K * 8"
- note added: "- leviathan header for draft stage - aiming for 20-30 pin - need to work out what is needed"
- note added: "- sd can consume around 100mA - current limit somehow - or add a shutdown - need to consider if this is same SPI bus as the debug card - programming this looks horrible"
- note added: "- some dumbass WILL somehow plug in a USB C the wrong way around otherwise - note D+/D- are differential - watch routing so this doesnt become impossible to solder"
- note added: "- super small jtag header - if no space boot becomes pads - and rsts will be connected - if thats a thing i can do idk"
- note added: "- will need to add a second i2c bus for debug card - route bus with care to avoid excess load"
- note added: "Clock"
- note added: "Debug Card Header"
- note added: "EEPROM"
- note added: "I2C Pullups"
- note added: "IMU"
- note added: "MCU"
- note added: "Programming"
- note added: "SD Card"
- note added: "Tempurature Sensor"
- note added: "USB-C Connector"
- note added: "Use if splitting GNDs"
- note removed: "Because: - Remove excess debug for space - Not needed during running - Using expansion slots debug can be accessed when needed - Faster clock, CANFD, IMU for future proofing - EEPROM for config flashing - Boot pad for space - Keeping jtag cuz goated - SD card for logging - temp sensor so board can have thermal shutoff/reg the h7/f7 do have internal ones but they r shit"
- note removed: "Planned changes: - higher clock - smaller JTAG header (6 pin micro) - remove 7 seg - remove uart - change to CANFD/-+58V fault compat can trancivers - add transient protection to can trancivers - add rs232/3rd can - add sd card - fix grounding - add pads for boot - smaller rst button - faster clock - add temp sensor - add imu? - add eeprom - add header for expansion slot with periherals and GPIO"
- moved on the sheet: J2, U1, U4
