File: CANna-VCU/vcu_proio.kicad_sch (KiCad schematic)
At the start: 0 parts

Commit message: first draft of full board
Parts:
- added #SP1: KP1600, symbol Device:Speaker
- added C49, C52: 1uF, Capacitor_SMD:C_0402_1005Metric, symbol Device:C_Small
- added C50, C51: 0.1uF, Capacitor_SMD:C_0402_1005Metric, symbol Device:C_Small
- added D14, D15, D16, D17, D18, D19, D20, D21: LED, LED_SMD:LED_0402_1005Metric, symbol Device:LED
- added J5: FSUK_RTD, Connector_PinHeader_2.54mm:PinHeader_1x02_P2.54mm_Vertical, symbol Connector_Generic:Conn_02x01
- added Q2, Q3, Q4, Q5, Q6, Q7, Q8: FDN359BN, Package_TO_SOT_SMD:SOT-23_Handsoldering, symbol SUFST:FDN359BN
- added R62, R63, R64, R65, R66, R67, R68, R69: 1.5K, Resistor_SMD:R_0402_1005Metric, symbol Device:R_Small
- added R70, R71, R72: 8.6K, Resistor_SMD:R_0402_1005Metric, symbol Device:R_Small
- added R73, R74, R81, R82, R83, R84: 0, Resistor_SMD:R_0402_1005Metric, symbol Device:R_Small
- added R75: 4.7K, Resistor_SMD:R_0402_1005Metric, symbol Device:R_Small
- added R76: 1k, Resistor_SMD:R_0402_1005Metric, symbol Device:R_Small
- added R77: 3k3, Resistor_SMD:R_0402_1005Metric, symbol Device:R_Small
- added R78, R79, R80, R85, R86, R87: 1K, Resistor_SMD:R_0402_1005Metric, symbol Device:R_Small
- added U10, U11, U12: 4504, Package_SO:SOIC-16W_5.3x10.2mm_P1.27mm, symbol 4xxx:4504
- added U9: ~, Package_DFN_QFN:TQFN-32-1EP_5x5mm_P0.5mm_EP3.1x3.1mm_ThermalVias, symbol SUFST:MAX22195
Connections:
- new net: R70.2, R71.1, U9.27 (EXTVM)
- new net: R65.1, U9.7 (IN4)
- new net: R62.1, U9.1 (IN1)
- new net: R63.1, U9.3 (IN2)
- new net: R82.1, R84.1, U12.16 (VDD)
- new net: D17.2 (A), U9.8 (LED4)
- new net: R81.1, R83.1, U11.16 (VDD)
- new net: D19.2 (A), U9.19 (LED6)
- new net: R73.1, R74.1, U10.1 (VCC)
- new net: J5.1 (Pin_1), Q2.3 (D), R76.1
- new net: Q8.3 (D), R87.1
- new net: Q4.3 (D), R79.1
- new net: R69.1, U9.24 (IN8)
- new net: Q5.3 (D), R80.1
- new net: R66.1, U9.18 (IN5)
- new net: D20.2 (A), U9.21 (LED7)
- new net: R64.1, U9.5 (IN3)
- new net: D14.2 (A), U9.2 (LED1)
- new net: R68.1, U9.22 (IN7)
- new net: D16.2 (A), U9.6 (LED3)
- new net: D18.2 (A), U9.17 (LED5)
- new net: R67.1, U9.20 (IN6)
- new net: D21.2 (A), U9.23 (LED8)
- new net: R72.1, U9.26 (REFDI)
- new net: D15.2 (A), U9.4 (LED2)
- new net: Q6.3 (D), R85.1
- new net: Q7.3 (D), R86.1
- new net: Q3.3 (D), R78.1
- new net +3V3: C51.2, C52.2, U10.16 (VDD), U11.1 (VCC), U12.1 (VCC), U9.28 (RDYEN), U9.31 (VDD3)
- new net +5V: R74.2, R81.2, R82.2
- new net +GLV_PROT: C49.2, C50.2, R70.1, R73.2, R83.2, R84.2, U9.30 (VDD24)
- new net GND: C49.1, C50.1, C51.1, C52.1, D14.1 (K), D15.1 (K), D16.1 (K), D17.1 (K), D18.1 (K), D19.1 (K), D20.1 (K), D21.1 (K), Q2.2 (S), Q3.2 (S), Q4.2 (S), Q5.2 (S), Q6.2 (S), Q7.2 (S), Q8.2 (S), R71.2, R72.2, R75.1, R77.1, U10.8 (VSS), U11.8 (VSS), U12.8 (VSS), U9.25 (GND), U9.32 (GND), U9.EX (GND)
- new net HSDI_GP1: R66.2
- new net HSDI_GP10: U10.14 (Fin)
- new net HSDI_GP2: R67.2
- new net HSDI_GP3: R68.2
- new net HSDI_GP4: R69.2
- new net HSDI_GP5: U10.3 (Ain)
- new net HSDI_GP6: U10.5 (Bin)
- new net HSDI_GP7: U10.7 (Cin)
- new net HSDI_GP8: U10.9 (Din)
- new net HSDI_GP9: U10.11 (Ein)
- new net HSDI_SCS1: R62.2
- new net HSDI_SCS2: R63.2
- new net HSDI_SCS3: R64.2
- new net HSDI_SCS4: R65.2
- new net HSDO_GP1: U11.12 (Eout)
- new net HSDO_GP2: U11.15 (Fout)
- new net HSDO_GP3: U12.2 (Aout)
- new net HSDO_GP4: U12.4 (Bout)
- new net HSDO_GP6: U12.6 (Cout)
- new net HSDO_GP7: U12.10 (Dout)
- new net HSDO_PWM1: U12.12 (Eout)
- new net HSDO_PWM2: U12.15 (Fout)
- new net HSDO_SCS1: U11.2 (Aout)
- new net HSDO_SCS2: U11.4 (Bout)
- new net HSDO_SCS3: U11.6 (Cout)
- new net HSDO_SCS4: U11.10 (Dout)
- new net LATCH_1: Q3.1 (G)
- new net LATCH_2: Q4.1 (G)
- new net LED_1: R78.2
- new net LED_2: R79.2
- new net LED_3: R80.2
- new net LED_4: R85.2
- new net LED_5: R86.2
- new net LED_6: R87.2
- new net LEVEL1_RDY: R75.2, U9.29 (READY)
- new net LSDI_GP1: U9.13 (OP5)
- new net LSDI_GP2: U9.14 (OP6)
- new net LSDI_GP3: U9.15 (OP7), U9.16 (OP8)
- new net LSDI_SCS1: U9.9 (OP1)
- new net LSDI_SCS10: U10.15 (Fout)
- new net LSDI_SCS2: U9.10 (OP2)
- new net LSDI_SCS3: U9.11 (OP3)
- new net LSDI_SCS4: U9.12 (OP4)
- new net LSDI_SCS5: U10.2 (Aout)
- new net LSDI_SCS6: U10.4 (Bout)
- new net LSDI_SCS7: U10.6 (Cout)
- new net LSDI_SCS8: U10.10 (Dout)
- new net LSDI_SCS9: U10.12 (Eout)
- new net LSDO_GP1: U11.11 (Ein)
- new net LSDO_GP2: U11.14 (Fin)
- new net LSDO_GP3: U12.3 (Ain)
- new net LSDO_GP4: U12.5 (Bin)
- new net LSDO_GP5: U12.7 (Cin)
- new net LSDO_GP6: U12.9 (Din)
- new net LSDO_PWM1: U12.11 (Ein)
- new net LSDO_PWM2: U12.14 (Fin)
- new net LSDO_SCS1: U11.3 (Ain)
- new net LSDO_SCS2: U11.5 (Bin)
- new net LSDO_SCS3: U11.7 (Cin)
- new net LSDO_SCS4: U11.9 (Din)
- new net LSD_LED_3: Q5.1 (G)
- new net LSD_LED_4: Q6.1 (G)
- new net LSD_LED_5: Q7.1 (G)
- new net LSD_LED_6: Q8.1 (G)
- new net LSD_R2D: Q2.1 (G), R77.2
- new net R2DS-: J5.2 (Pin_2), R76.2
- no-connect marks 0 -> 2
Other:
- note added: "**ADD PULLDOWNS**"
- note added: "**PLACEHOLDER** **NOT 24V COMPATIBLE**"
- note added: "All LED connections are current paths to ground via MOSFET, rather than a driving output Other side of LED should be connected to 12V, current limiting resistors here are optional (could be external)"
- note added: "Dash LEDs"
- note added: "FSUK requires >90dB so R = 0 FSG requires <90dB so R > 0?"
- note added: "HV In"
- note added: "IN"
- note added: "OUT"
- note added: "Pull to ground in case MCU disconnected"
- note added: "R2D"
- note added: "VC_LEDS provides a connection to ground for 2s on start up This is used to meet T11.9.5("visual check")"
- note added: "Var Voltage In"
- note added: "Var Voltage Out"
- note removed: "Planned changes: - check if optoiso is the best choice - swap for a much smaller package - double number of inputs Why: - future proofing - space will be an issue on this board, so trying to keep things neat"
- note removed: "Planned changes: - double output channels and intergrate with fet array on main - decide if to use fets or optoisos - could have all the same or low speed and high speed options - might add 5v input capabilities Because: - channels can be multipurpose - space saving - switching speed"
