File: CANna-VCU/CANna-VCU.kicad_pcb (KiCad board)
At the start: 2 copper layers, 100 x 70 mm, 77 parts, among them J11 PWR, J8 OUT, J9 USB_C_Receptacle_USB2.0_16P, SW1 SW_Push, U1 TCAN3400-Q1, U11 LMR33630CDDA, U12 LD1117S33TR_SOT223, U2 TCAN3400-Q1, U3 M24256-DRD, U4 TLV274, U6 STM32F746ZGT6

Commit message: first draft of full board
Parts:
- removed C63, C64: 100n, Capacitor_SMD:C_0805_2012Metric_Pad1.18x1.45mm_HandSolder
- removed C65: 4.7n, Capacitor_SMD:C_0805_2012Metric_Pad1.18x1.45mm_HandSolder
- removed the H1 at (122.0, 113.0)
- removed the H1 at (208.0, 57.0)
- removed the H1 at (208.0, 113.0)
- removed the H1 at (122.0, 57.0)
- removed J11: PWR, Connector_Molex:Molex_Micro-Fit_3.0_43045-0400_2x02_P3.00mm_Horizontal
- removed J8: OUT, Connector_Molex:Molex_Micro-Fit_3.0_43045-0800_2x04_P3.00mm_Horizontal
- removed the R10 at (67.6, 116.3)
- removed the R11 at (67.6, 119.2)
- removed the U1 at (61.0, 112.3)
- added C10: 4.7uF, Capacitor_SMD:C_0402_1005Metric, F.Cu at (49.5, 68.6)
- added C11: 100nF, Capacitor_SMD:C_0402_1005Metric, F.Cu at (49.5, 70.6)
- added C12: 100nF, Capacitor_SMD:C_0402_1005Metric, F.Cu at (49.5, 72.6)
- added C13: 100nF, Capacitor_SMD:C_0402_1005Metric, F.Cu at (52.4, 66.7)
- added C14: 2.2u, Capacitor_SMD:C_0805_2012Metric_Pad1.18x1.45mm_HandSolder, F.Cu at (62.9, 67.2)
- added C15: 100nF, Capacitor_SMD:C_0603_1608Metric, F.Cu at (72.4, 71.1)
- added C16: 2.2u, Capacitor_SMD:C_0805_2012Metric_Pad1.18x1.45mm_HandSolder, F.Cu at (62.9, 70.2)
- added C17: 100nF, Capacitor_SMD:C_0402_1005Metric, F.Cu at (52.4, 68.6)
- added C18: 100nF, Capacitor_SMD:C_0402_1005Metric, F.Cu at (52.4, 70.6)
- added C19: 1uF, Capacitor_SMD:C_0402_1005Metric, F.Cu at (52.4, 72.6)
- added C21: 10uF, Capacitor_SMD:C_0402_1005Metric, F.Cu at (93.8, 58.1)
- added C39: 100n, Capacitor_SMD:C_0402_1005Metric, F.Cu at (83.6, 90.5)
- added C4: 100nF, Capacitor_SMD:C_0402_1005Metric, F.Cu at (43.8, 72.6)
- added C40: 100n, Capacitor_SMD:C_0402_1005Metric, F.Cu at (83.6, 92.4)
- added C41: 100n, Capacitor_SMD:C_0402_1005Metric, F.Cu at (83.6, 94.4)
- added C42: 100n, Capacitor_SMD:C_0402_1005Metric, F.Cu at (86.5, 90.5)
- added C43: 1n, Capacitor_SMD:C_0402_1005Metric, F.Cu at (86.5, 92.4)
- added C44: 1n, Capacitor_SMD:C_0402_1005Metric, F.Cu at (86.5, 94.4)
- added C45: 1n, Capacitor_SMD:C_0402_1005Metric, F.Cu at (89.3, 90.5)
- added C46: 1n, Capacitor_SMD:C_0402_1005Metric, F.Cu at (89.3, 92.4)
- added C47: 100n, Capacitor_SMD:C_0402_1005Metric, F.Cu at (89.3, 94.4)
- added C49: 1uF, Capacitor_SMD:C_0402_1005Metric, F.Cu at (65.0, 88.3)
- added C5: 100n, Capacitor_SMD:C_0402_1005Metric, F.Cu at (46.6, 66.7)
- added C50: 0.1uF, Capacitor_SMD:C_0402_1005Metric, F.Cu at (65.0, 90.3)
- added C51: 0.1uF, Capacitor_SMD:C_0402_1005Metric, F.Cu at (65.0, 92.2)
- added C52: 1uF, Capacitor_SMD:C_0402_1005Metric, F.Cu at (65.0, 94.2)
- added C53: 100n, Capacitor_SMD:C_0402_1005Metric, F.Cu at (93.8, 63.3)
- added C54: 100n, Capacitor_SMD:C_0402_1005Metric, F.Cu at (93.8, 65.2)
- added C55: 4.7n, Capacitor_SMD:C_0402_1005Metric, F.Cu at (93.8, 67.2)
- added C56: 4.7n, Capacitor_SMD:C_0402_1005Metric, F.Cu at (93.8, 69.2)
- added C6: 100n, Capacitor_SMD:C_0402_1005Metric, F.Cu at (46.6, 68.6)
- added C7: 4.7pF, Capacitor_SMD:C_0402_1005Metric, F.Cu at (46.6, 70.6)
- added C8: 4.7pF, Capacitor_SMD:C_0402_1005Metric, F.Cu at (46.6, 72.6)
- added C9: 100nF, Capacitor_SMD:C_0402_1005Metric, F.Cu at (49.5, 66.7)
- added D10: BZX84-C3V3, Package_TO_SOT_SMD:SOT-23, F.Cu at (96.2, 78.0)
- added D11: BZX84-C3V3, Package_TO_SOT_SMD:SOT-23, F.Cu at (96.2, 82.6)
- added D12: BZX84-C3V3, Package_TO_SOT_SMD:SOT-23, F.Cu at (96.2, 87.2)
- added D13: BZX84-C3V3, Package_TO_SOT_SMD:SOT-23, F.Cu at (96.2, 91.8)
- added D14: LED, LED_SMD:LED_0402_1005Metric, F.Cu at (50.5, 88.3)
- added D15: LED, LED_SMD:LED_0402_1005Metric, F.Cu at (50.5, 90.3)
- added D16: LED, LED_SMD:LED_0402_1005Metric, F.Cu at (50.5, 92.3)
- added D17: LED, LED_SMD:LED_0402_1005Metric, F.Cu at (50.5, 94.3)
- added D18: LED, LED_SMD:LED_0402_1005Metric, F.Cu at (50.5, 96.3)
- added D19: LED, LED_SMD:LED_0402_1005Metric, F.Cu at (50.5, 98.3)
- added D2: BZX84Cxx, Package_TO_SOT_SMD:SOT-23, F.Cu at (92.8, 52.7)
- added D20: LED, LED_SMD:LED_0402_1005Metric, F.Cu at (50.5, 100.3)
- added D21: LED, LED_SMD:LED_0402_1005Metric, F.Cu at (50.5, 102.2)
- added D3: D_Schottky, Diode_SMD:D_0603_1608Metric, F.Cu at (90.3, 56.4)
- added D4: D_Schottky, Diode_SMD:D_0603_1608Metric, F.Cu at (90.3, 59.0)
- added F1: 500mA, Fuse:Fuse_0603_1608Metric, F.Cu at (86.0, 58.9)
- added H1: M3, MountingHole:MountingHole_3.2mm_M3, F.Cu at (87.9, 36.4)
- added H2: M3, MountingHole:MountingHole_3.2mm_M3, F.Cu at (87.9, 44.4)
- added H3: M3, MountingHole:MountingHole_3.2mm_M3, F.Cu at (95.9, 36.4)
- added H4: M3, MountingHole:MountingHole_3.2mm_M3, F.Cu at (95.9, 44.4)
- added J3: SD_Card_Device, Connector_Card:SD_Hirose_DM1AA_SF_PEJ82, F.Cu at (58.9, 49.4)
- added J5: FSUK_RTD, Connector_PinHeader_2.54mm:PinHeader_1x02_P2.54mm_Vertical, F.Cu at (76.0, 89.6)
- added L1: L, Inductor_SMD:L_0603_1608Metric_Pad1.05x0.95mm_HandSolder, F.Cu at (86.1, 56.4)
- added Q1: FDN359BN, Package_TO_SOT_SMD:SOT-23_Handsoldering, F.Cu at (87.2, 52.8)
- added Q2: FDN359BN, Package_TO_SOT_SMD:SOT-23_Handsoldering, F.Cu at (45.6, 78.1)
- added Q3: FDN359BN, Package_TO_SOT_SMD:SOT-23_Handsoldering, F.Cu at (45.6, 82.8)
- added Q4: FDN359BN, Package_TO_SOT_SMD:SOT-23_Handsoldering, F.Cu at (45.6, 87.6)
- added Q5: FDN359BN, Package_TO_SOT_SMD:SOT-23_Handsoldering, F.Cu at (45.6, 92.4)
- added Q6: FDN359BN, Package_TO_SOT_SMD:SOT-23_Handsoldering, F.Cu at (45.6, 97.2)
- added Q7: FDN359BN, Package_TO_SOT_SMD:SOT-23_Handsoldering, F.Cu at (45.6, 101.9)
- added Q8: FDN359BN, Package_TO_SOT_SMD:SOT-23_Handsoldering, F.Cu at (45.6, 106.7)
- added R3: 100K, Resistor_SMD:R_0402_1005Metric, F.Cu at (76.8, 37.4)
- added R38: 100k, Resistor_SMD:R_0402_1005Metric, F.Cu at (83.6, 76.5)
- added R39: 100k, Resistor_SMD:R_0402_1005Metric, F.Cu at (83.6, 78.5)
- added R4: 1.3K, Resistor_SMD:R_0402_1005Metric, F.Cu at (76.8, 39.4)
- added R40: 100k, Resistor_SMD:R_0402_1005Metric, F.Cu at (83.6, 80.5)
- added R41: 100k, Resistor_SMD:R_0402_1005Metric, F.Cu at (83.6, 82.5)
- added R42: 1k, Resistor_SMD:R_0402_1005Metric, F.Cu at (83.6, 84.5)
- added R43: 1k, Resistor_SMD:R_0402_1005Metric, F.Cu at (83.6, 86.5)
- added R44: 1k, Resistor_SMD:R_0402_1005Metric, F.Cu at (83.6, 88.5)
- added R45: 1k, Resistor_SMD:R_0402_1005Metric, F.Cu at (86.5, 76.5)
- added R46: 75k, Resistor_SMD:R_0402_1005Metric, F.Cu at (86.5, 78.5)
- added R47: 5.6k, Resistor_SMD:R_0402_1005Metric, F.Cu at (86.5, 80.5)
- added R48: 5.6k, Resistor_SMD:R_0402_1005Metric, F.Cu at (86.5, 82.5)
- added R49: 1.8k, Resistor_SMD:R_0402_1005Metric, F.Cu at (86.5, 84.5)
- added R5: 10K, Resistor_SMD:R_0402_1005Metric, F.Cu at (76.8, 41.4)
- added R50: 75k, Resistor_SMD:R_0402_1005Metric, F.Cu at (86.5, 86.5)
- added R51: 5.6k, Resistor_SMD:R_0402_1005Metric, F.Cu at (86.5, 88.5)
- added R52: 5.6k, Resistor_SMD:R_0402_1005Metric, F.Cu at (89.4, 76.5)
- added R53: 1.8k, Resistor_SMD:R_0402_1005Metric, F.Cu at (89.4, 78.5)
- added R54: 75k, Resistor_SMD:R_0402_1005Metric, F.Cu at (89.4, 80.5)
- added R55: 5.6k, Resistor_SMD:R_0402_1005Metric, F.Cu at (89.4, 82.5)
- added R56: 5.6k, Resistor_SMD:R_0402_1005Metric, F.Cu at (89.4, 84.5)
- added R57: 1.8k, Resistor_SMD:R_0402_1005Metric, F.Cu at (89.4, 86.5)
- added R58: 75k, Resistor_SMD:R_0402_1005Metric, F.Cu at (89.4, 88.5)
- added R59: 5.6k, Resistor_SMD:R_0402_1005Metric, F.Cu at (92.3, 76.5)
- added R6: 10K, Resistor_SMD:R_0402_1005Metric, F.Cu at (76.8, 43.4)
- added R60: 5.6k, Resistor_SMD:R_0402_1005Metric, F.Cu at (92.3, 78.5)
- added R61: 1.8k, Resistor_SMD:R_0402_1005Metric, F.Cu at (92.3, 80.5)
- added R62: 1.5K, Resistor_SMD:R_0402_1005Metric, F.Cu at (53.4, 88.3)
- added R63: 1.5K, Resistor_SMD:R_0402_1005Metric, F.Cu at (53.4, 90.3)
- added R64: 1.5K, Resistor_SMD:R_0402_1005Metric, F.Cu at (53.4, 92.3)
- added R65: 1.5K, Resistor_SMD:R_0402_1005Metric, F.Cu at (53.4, 94.3)
- added R66: 1.5K, Resistor_SMD:R_0402_1005Metric, F.Cu at (53.4, 96.3)
- added R67: 1.5K, Resistor_SMD:R_0402_1005Metric, F.Cu at (53.4, 98.3)
- added R68: 1.5K, Resistor_SMD:R_0402_1005Metric, F.Cu at (53.4, 100.3)
- added R69: 1.5K, Resistor_SMD:R_0402_1005Metric, F.Cu at (56.3, 88.3)
- added R7: 2.2K, Resistor_SMD:R_0402_1005Metric, F.Cu at (76.8, 45.4)
- added R70: 8.6K, Resistor_SMD:R_0402_1005Metric, F.Cu at (56.3, 90.3)
- added R71: 8.6K, Resistor_SMD:R_0402_1005Metric, F.Cu at (56.3, 92.3)
- added R72: 8.6K, Resistor_SMD:R_0402_1005Metric, F.Cu at (56.3, 94.3)
- added R73: 0, Resistor_SMD:R_0402_1005Metric, F.Cu at (56.3, 96.3)
- added R74: 0, Resistor_SMD:R_0402_1005Metric, F.Cu at (56.3, 98.3)
- added R75: 4.7K, Resistor_SMD:R_0402_1005Metric, F.Cu at (56.3, 100.3)
- added R76: 1k, Resistor_SMD:R_0402_1005Metric, F.Cu at (59.2, 88.3)
- added R77: 3k3, Resistor_SMD:R_0402_1005Metric, F.Cu at (59.2, 90.3)
- added R78: 1K, Resistor_SMD:R_0402_1005Metric, F.Cu at (59.2, 92.3)
- added R79: 1K, Resistor_SMD:R_0402_1005Metric, F.Cu at (59.2, 94.3)
- added R8: 2.2K, Resistor_SMD:R_0402_1005Metric, F.Cu at (76.8, 47.4)
- added R80: 1K, Resistor_SMD:R_0402_1005Metric, F.Cu at (59.2, 96.3)
- added R81: 0, Resistor_SMD:R_0402_1005Metric, F.Cu at (59.2, 98.3)
- added R82: 0, Resistor_SMD:R_0402_1005Metric, F.Cu at (59.2, 100.3)
- added R83: 0, Resistor_SMD:R_0402_1005Metric, F.Cu at (62.1, 88.3)
- added R84: 0, Resistor_SMD:R_0402_1005Metric, F.Cu at (62.1, 90.3)
- added R85: 1K, Resistor_SMD:R_0402_1005Metric, F.Cu at (62.1, 92.3)
- added R86: 1K, Resistor_SMD:R_0402_1005Metric, F.Cu at (62.1, 94.3)
- added R87: 1K, Resistor_SMD:R_0402_1005Metric, F.Cu at (62.1, 96.3)
- added R88: 60R, Resistor_SMD:R_0402_1005Metric, F.Cu at (90.9, 63.3)
- added R89: 60R, Resistor_SMD:R_0402_1005Metric, F.Cu at (90.9, 65.3)
- added R9: 100k, Resistor_SMD:R_0402_1005Metric, F.Cu at (93.8, 56.1)
- added R90: 60R, Resistor_SMD:R_0402_1005Metric, F.Cu at (90.9, 67.2)
- added R91: 60R, Resistor_SMD:R_0402_1005Metric, F.Cu at (90.9, 69.2)
- added SW2: CK_KMS2xxG, Button_Switch_SMD:SW_SPST_CK_KMS2xxGP, F.Cu at (78.7, 56.2)
- added U10: 4504, Package_SO:SOIC-16W_5.3x10.2mm_P1.27mm, F.Cu at (54.0, 81.5)
- added U11: 4504, Package_SO:SOIC-16W_5.3x10.2mm_P1.27mm, F.Cu at (64.5, 81.5)
- added U12: 4504, Package_SO:SOIC-16W_5.3x10.2mm_P1.27mm, F.Cu at (74.9, 81.5)
- added U13: LTC2875-DD, Package_DFN_QFN:DFN-8-1EP_3x3mm_P0.5mm_EP1.66x2.38mm, F.Cu at (86.9, 64.6)
- added U14: LTC2875-DD, Package_DFN_QFN:DFN-8-1EP_3x3mm_P0.5mm_EP1.66x2.38mm, F.Cu at (86.9, 69.2)
- added U3: ISM330DHCX, Package_LGA:LGA-14_3x2.5mm_P0.5mm_LayoutBorder3x4y, F.Cu at (72.7, 67.8)
- added U8: TLV274, Package_SO:SOIC-14_3.9x8.7mm_P1.27mm, F.Cu at (102.9, 80.8)
- added U9: ~, Package_DFN_QFN:TQFN-32-1EP_5x5mm_P0.5mm_EP3.1x3.1mm_ThermalVias, F.Cu at (70.1, 91.0)
- added Y1: 25MHz, Crystal:Crystal_SMD_3225-4Pin_3.2x2.5mm_HandSoldering, F.Cu at (57.1, 68.5)
- C1: value 100n -> 0.1uF; footprint Capacitor_SMD:C_0805_2012Metric_Pad1.18x1.45mm_HandSolder -> Capacitor_SMD:C_0402_1005Metric
- C2: value 100n -> 10uF; footprint Capacitor_SMD:C_0805_2012Metric_Pad1.18x1.45mm_HandSolder -> Capacitor_SMD:C_0402_1005Metric
- C20: renamed from C35; footprint Capacitor_SMD:C_0603_1608Metric -> Capacitor_SMD:C_0402_1005Metric
- C22: renamed from C36; footprint Capacitor_SMD:C_0603_1608Metric -> Capacitor_SMD:C_0402_1005Metric
- C23: renamed from C37; footprint Capacitor_SMD:C_0603_1608Metric -> Capacitor_SMD:C_0402_1005Metric
- C24: renamed from C38; footprint Capacitor_SMD:C_0603_1608Metric -> Capacitor_SMD:C_0402_1005Metric
- C25: renamed from C39; footprint Capacitor_SMD:C_0603_1608Metric -> Capacitor_SMD:C_0402_1005Metric
- C26: renamed from C40; footprint Capacitor_SMD:C_0603_1608Metric -> Capacitor_SMD:C_0402_1005Metric
- C27: renamed from C41; footprint Capacitor_SMD:C_0603_1608Metric -> Capacitor_SMD:C_0402_1005Metric
- C28: renamed from C42; footprint Capacitor_SMD:C_0603_1608Metric -> Capacitor_SMD:C_0402_1005Metric
- C29: renamed from C43; footprint Capacitor_SMD:C_0805_2012Metric_Pad1.18x1.45mm_HandSolder -> Capacitor_SMD:C_0402_1005Metric
- C3: value 4.7n -> 68nF; footprint Capacitor_SMD:C_0805_2012Metric_Pad1.18x1.45mm_HandSolder -> Capacitor_SMD:C_0402_1005Metric
- C30: renamed from C44; footprint Capacitor_SMD:C_0805_2012Metric_Pad1.18x1.45mm_HandSolder -> Capacitor_SMD:C_0402_1005Metric
- C31: renamed from C4; footprint Capacitor_SMD:C_0805_2012Metric_Pad1.18x1.45mm_HandSolder -> Capacitor_SMD:C_0402_1005Metric
- C32: renamed from C5; footprint Capacitor_SMD:C_0805_2012Metric_Pad1.18x1.45mm_HandSolder -> Capacitor_SMD:C_0402_1005Metric
- C33: renamed from C6; footprint Capacitor_SMD:C_0805_2012Metric_Pad1.18x1.45mm_HandSolder -> Capacitor_SMD:C_0402_1005Metric
- C34: renamed from C7; footprint Capacitor_SMD:C_0805_2012Metric_Pad1.18x1.45mm_HandSolder -> Capacitor_SMD:C_0402_1005Metric
- C35: renamed from C8; footprint Capacitor_SMD:C_0805_2012Metric_Pad1.18x1.45mm_HandSolder -> Capacitor_SMD:C_0402_1005Metric
- C36: renamed from C9; footprint Capacitor_SMD:C_0805_2012Metric_Pad1.18x1.45mm_HandSolder -> Capacitor_SMD:C_0402_1005Metric
- C37: renamed from C10; footprint Capacitor_SMD:C_0805_2012Metric_Pad1.18x1.45mm_HandSolder -> Capacitor_SMD:C_0402_1005Metric
- C38: renamed from C11; footprint Capacitor_SMD:C_0805_2012Metric_Pad1.18x1.45mm_HandSolder -> Capacitor_SMD:C_0402_1005Metric
- C48: renamed from C12; footprint Capacitor_SMD:C_0805_2012Metric_Pad1.18x1.45mm_HandSolder -> Capacitor_SMD:C_0402_1005Metric
- R1, R2: value 60R -> 5.1k; footprint Resistor_SMD:R_0805_2012Metric_Pad1.20x1.40mm_HandSolder -> Resistor_SMD:R_0402_1005Metric
- R10: renamed from R82; footprint Resistor_SMD:R_0603_1608Metric -> Resistor_SMD:R_0402_1005Metric
- R11: renamed from R83; footprint Resistor_SMD:R_0603_1608Metric -> Resistor_SMD:R_0402_1005Metric
- R12: renamed from R84; footprint Resistor_SMD:R_0603_1608Metric -> Resistor_SMD:R_0402_1005Metric
- R13: renamed from R85; footprint Resistor_SMD:R_0805_2012Metric_Pad1.20x1.40mm_HandSolder -> Resistor_SMD:R_0402_1005Metric
- R14: renamed from R12; footprint Resistor_SMD:R_0805_2012Metric_Pad1.20x1.40mm_HandSolder -> Resistor_SMD:R_0402_1005Metric
- R15: renamed from R13; footprint Resistor_SMD:R_0805_2012Metric_Pad1.20x1.40mm_HandSolder -> Resistor_SMD:R_0402_1005Metric
- R16: renamed from R14; footprint Resistor_SMD:R_0805_2012Metric_Pad1.20x1.40mm_HandSolder -> Resistor_SMD:R_0402_1005Metric
- R17: renamed from R15; footprint Resistor_SMD:R_0805_2012Metric_Pad1.20x1.40mm_HandSolder -> Resistor_SMD:R_0402_1005Metric
- R18: renamed from R16; footprint Resistor_SMD:R_0805_2012Metric_Pad1.20x1.40mm_HandSolder -> Resistor_SMD:R_0402_1005Metric
- R19: renamed from R17; footprint Resistor_SMD:R_0805_2012Metric_Pad1.20x1.40mm_HandSolder -> Resistor_SMD:R_0402_1005Metric
- R20: renamed from R18; footprint Resistor_SMD:R_0805_2012Metric_Pad1.20x1.40mm_HandSolder -> Resistor_SMD:R_0402_1005Metric
- R21: renamed from R19; footprint Resistor_SMD:R_0805_2012Metric_Pad1.20x1.40mm_HandSolder -> Resistor_SMD:R_0402_1005Metric
- R22: renamed from R20; footprint Resistor_SMD:R_0805_2012Metric_Pad1.20x1.40mm_HandSolder -> Resistor_SMD:R_0402_1005Metric
- R23: renamed from R21; footprint Resistor_SMD:R_0805_2012Metric_Pad1.20x1.40mm_HandSolder -> Resistor_SMD:R_0402_1005Metric
- R24: renamed from R22; footprint Resistor_SMD:R_0805_2012Metric_Pad1.20x1.40mm_HandSolder -> Resistor_SMD:R_0402_1005Metric
- R25: renamed from R23; footprint Resistor_SMD:R_0805_2012Metric_Pad1.20x1.40mm_HandSolder -> Resistor_SMD:R_0402_1005Metric
- R26: renamed from R24; footprint Resistor_SMD:R_0805_2012Metric_Pad1.20x1.40mm_HandSolder -> Resistor_SMD:R_0402_1005Metric
- R27: renamed from R25; footprint Resistor_SMD:R_0805_2012Metric_Pad1.20x1.40mm_HandSolder -> Resistor_SMD:R_0402_1005Metric
- R28: renamed from R26; footprint Resistor_SMD:R_0805_2012Metric_Pad1.20x1.40mm_HandSolder -> Resistor_SMD:R_0402_1005Metric
- R29: renamed from R27; footprint Resistor_SMD:R_0805_2012Metric_Pad1.20x1.40mm_HandSolder -> Resistor_SMD:R_0402_1005Metric
- R30: renamed from R28; footprint Resistor_SMD:R_0805_2012Metric_Pad1.20x1.40mm_HandSolder -> Resistor_SMD:R_0402_1005Metric
- R31: renamed from R29; footprint Resistor_SMD:R_0805_2012Metric_Pad1.20x1.40mm_HandSolder -> Resistor_SMD:R_0402_1005Metric
- R32: renamed from R30; footprint Resistor_SMD:R_0805_2012Metric_Pad1.20x1.40mm_HandSolder -> Resistor_SMD:R_0402_1005Metric
- R33: renamed from R31; footprint Resistor_SMD:R_0805_2012Metric_Pad1.20x1.40mm_HandSolder -> Resistor_SMD:R_0402_1005Metric
- R34: renamed from R32; footprint Resistor_SMD:R_0805_2012Metric_Pad1.20x1.40mm_HandSolder -> Resistor_SMD:R_0402_1005Metric
- R35: renamed from R33; footprint Resistor_SMD:R_0805_2012Metric_Pad1.20x1.40mm_HandSolder -> Resistor_SMD:R_0402_1005Metric
- R36: renamed from R34; footprint Resistor_SMD:R_0805_2012Metric_Pad1.20x1.40mm_HandSolder -> Resistor_SMD:R_0402_1005Metric
- R37: renamed from R35; footprint Resistor_SMD:R_0805_2012Metric_Pad1.20x1.40mm_HandSolder -> Resistor_SMD:R_0402_1005Metric
- SW1: value SW_Push -> CK_KMS2xxG; footprint Button_Switch_THT:SW_PUSH_6mm -> Button_Switch_SMD:SW_SPST_CK_KMS2xxGP
- U2: value TCAN3400-Q1 -> MCP9800Ax-xOT; footprint Package_SO:SOIC-8_3.9x4.9mm_P1.27mm -> Package_TO_SOT_SMD:SOT-23-5
- moved R2 78.5 mm to (76.8, 35.4)
- moved R1 77.5 mm to (76.8, 33.4)
- moved U2 51.2 mm to (67.8, 68.1)
- moved SW1 48.5 mm to (78.7, 50.8)
- moved C3 47.1 mm to (43.8, 70.6)
- moved C2 46.0 mm to (43.8, 68.6)
- moved C1 45.0 mm to (43.8, 66.7)
- moved C30 33.6 mm to (83.2, 155.2)
- moved R13 33.6 mm to (87.9, 155.2)
- moved U6 33.6 mm to (85.7, 140.0)
- moved C22 33.6 mm to (74.7, 139.5)
- moved C23 33.6 mm to (74.7, 142.0)
- moved C25 33.6 mm to (74.7, 147.1)
- moved C26 33.6 mm to (74.7, 149.6)
- moved C28 33.6 mm to (78.7, 139.5)
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- renumbered D11 to D5, D1 to D6, D2 to D7, D3 to D8, D4 to D9, J9 to J2, U3 to U1, U6 to U4, U11 to U5, U12 to U6, U4 to U7
Connections:
- net Net-(J9-VBUS-PadA4) renamed +5V_UNPROT
- C1 pad 2: Net-(U1-SHDN) -> +3V3
- C20 pad 1: +12V -> +GLV_PROT
- C22 pad 1: +12V -> +GLV_PROT
- C3 pad 1: Net-(C3-Pad1) -> GND
- C3 pad 2: GND -> /MCU/nRST
- J2 pad A1: Net-(J9-GND-PadA1) -> GND
- J2 pad A12: Net-(J9-GND-PadA1) -> GND
- J2 pad A5: unconnected-(J9-CC1-PadA5) -> Net-(J2-CC1)
- J2 pad A6: unconnected-(J9-D+-PadA6) -> /MCU/USB_D+
- J2 pad A7: unconnected-(J9-D--PadA7) -> /MCU/USB_D-
- J2 pad B1: Net-(J9-GND-PadA1) -> GND
- J2 pad B12: Net-(J9-GND-PadA1) -> GND
- J2 pad B5: unconnected-(J9-CC2-PadB5) -> Net-(J2-CC2)
- J2 pad B6: unconnected-(J9-D+-PadB6) -> /MCU/USB_D+
- J2 pad B7: unconnected-(J9-D--PadB7) -> /MCU/USB_D-
- J2 pad S1: unconnected-(J9-SHIELD-PadS1) -> GND
- R1 pad 1: Net-(C3-Pad1) -> GND
- R1 pad 2: 2_CANH -> Net-(J2-CC1)
- R2 pad 1: 2_CANL -> GND
- R2 pad 2: Net-(C3-Pad1) -> Net-(J2-CC2)
- SW1 pad 1: (no net) -> +3V3
- SW1 pad 2: (no net) -> GND
- U1 pad 1: unconnected-(U3-E0-Pad1) -> +3V3
- U1 pad 2: unconnected-(U3-E1-Pad2) -> +3V3
- U1 pad 3: unconnected-(U3-E2-Pad3) -> +3V3
- U1 pad 4: unconnected-(U3-VSS-Pad4) -> GND
- U1 pad 5: unconnected-(U3-SDA-Pad5) -> /MCU/I2C_SDA
- U1 pad 6: unconnected-(U3-SCL-Pad6) -> /MCU/I2C_SCL
- U1 pad 7: unconnected-(U3-WC-Pad7) -> /MCU/EEPROM_WC
- U1 pad 8: unconnected-(U3-VCC-Pad8) -> +3V3
- U2 pad 1: MCU_CAN2_TX -> +3V3
- U2 pad 3: +3V3 -> /MCU/TOO_HOT
- U2 pad 4: MCU_CAN2_RX -> /MCU/I2C_CLK
- U2 pad 5: Net-(U2-SHDN) -> /MCU/I2C_SDA
- U4 pad 100: unconnected-(U6-PA8-Pad100) -> /MCU/UART_CLK
- U4 pad 101: unconnected-(U6-PA9-Pad101) -> /MCU/UART_TX
- U4 pad 102: unconnected-(U6-PA10-Pad102) -> /MCU/UART_RX
- U4 pad 103: unconnected-(U6-PA11-Pad103) -> /MCU/USB_D-
- U4 pad 104: unconnected-(U6-PA12-Pad104) -> /MCU/USB_D+
- U4 pad 105: unconnected-(U6-PA13-Pad105) -> /MCU/SWDIO
- U4 pad 106: unconnected-(U6-VCAP_2-Pad106) -> Net-(U4-VCAP_2)
- U4 pad 107: Net-(U6-VSS-Pad107) -> GND
- U4 pad 108: unconnected-(U6-VDD-Pad108) -> +3V3
- U4 pad 109: unconnected-(U6-PA14-Pad109) -> /MCU/SWCLK
- U4 pad 114: unconnected-(U6-PD0-Pad114) -> /MCU/CAN0_RX
- U4 pad 115: unconnected-(U6-PD1-Pad115) -> /MCU/CAN0_TX
- U4 pad 120: Net-(U6-VSS-Pad107) -> GND
- U4 pad 121: unconnected-(U6-VDD-Pad121) -> +3V3
- U4 pad 130: Net-(U6-VSS-Pad107) -> GND
- U4 pad 131: unconnected-(U6-VDD-Pad131) -> +3V3
- U4 pad 133: unconnected-(U6-PB3-Pad133) -> /MCU/SWO
- U4 pad 134: unconnected-(U6-PB4-Pad134) -> /MCU/nRST
- U4 pad 136: unconnected-(U6-PB6-Pad136) -> /MCU/CAN1_TX
- U4 pad 138: unconnected-(U6-BOOT0-Pad138) -> /MCU/BOOT_0
- U4 pad 139: unconnected-(U6-PB8-Pad139) -> /MCU/I2C_SCL
- U4 pad 140: unconnected-(U6-PB9-Pad140) -> /MCU/I2C_SDA
- U4 pad 144: unconnected-(U6-VDD-Pad144) -> +3V3
- U4 pad 16: Net-(U6-VSS-Pad107) -> GND
- U4 pad 17: unconnected-(U6-VDD-Pad17) -> +3V3
- U4 pad 23: unconnected-(U6-PH0-Pad23) -> /MCU/OSC_IN
- U4 pad 24: unconnected-(U6-PH1-Pad24) -> /MCU/OSC_OUT
- U4 pad 25: unconnected-(U6-NRST-Pad25) -> /MCU/RST
- U4 pad 30: unconnected-(U6-VDD-Pad30) -> +3V3
- U4 pad 31: unconnected-(U6-VSSA-Pad31) -> GND
- U4 pad 33: unconnected-(U6-VDDA-Pad33) -> +3V3A
- U4 pad 38: Net-(U6-VSS-Pad107) -> GND
- U4 pad 39: unconnected-(U6-VDD-Pad39) -> +3V3
- U4 pad 51: Net-(U6-VSS-Pad107) -> GND
- U4 pad 52: unconnected-(U6-VDD-Pad52) -> +3V3
- U4 pad 6: unconnected-(U6-VBAT-Pad6) -> +3V3
- U4 pad 61: Net-(U6-VSS-Pad107) -> GND
- U4 pad 62: unconnected-(U6-VDD-Pad62) -> +3V3
- U4 pad 71: unconnected-(U6-VCAP_1-Pad71) -> Net-(U4-VCAP_1)
- U4 pad 72: unconnected-(U6-VDD-Pad72) -> +3V3
- U4 pad 73: unconnected-(U6-PB12-Pad73) -> /MCU/CAN1_RX
- U4 pad 83: Net-(U6-VSS-Pad107) -> GND
- U4 pad 84: unconnected-(U6-VDD-Pad84) -> +3V3
- U4 pad 94: Net-(U6-VSS-Pad107) -> GND
- U4 pad 95: unconnected-(U6-VDDUSB-Pad95) -> +3V3
- U5 pad 2: +12V -> +GLV_PROT
- U5 pad 3: +12V -> +GLV_PROT

Commit message: tidying up
Parts:
- added REF**: Harwin_LTek-Male_2x22_P2.00mm_Vertical_StrainRelief, Connector_Harwin:Harwin_LTek-Male_2x22_P2.00mm_Vertical_StrainRelief, F.Cu at (225.5, 61.0)

Commit message: added power managment bits
Parts:
- removed the REF** at (225.5, 61.0)
- added C54: 100n, Capacitor_SMD:C_0402_1005Metric, F.Cu at (129.7, 77.5)
- added C56: 4.7n, Capacitor_SMD:C_0402_1005Metric, F.Cu at (123.1, 77.4)
- added D14: LED, LED_SMD:LED_0402_1005Metric, F.Cu at (176.5, 71.2)
- added D15: LED, LED_SMD:LED_0402_1005Metric, F.Cu at (176.5, 69.8)
- added D16: LED, LED_SMD:LED_0402_1005Metric, F.Cu at (176.5, 68.2)
- added D17: LED, LED_SMD:LED_0402_1005Metric, F.Cu at (176.5, 66.8)
- added D18: LED, LED_SMD:LED_0402_1005Metric, F.Cu at (176.5, 65.2)
- added D19: LED, LED_SMD:LED_0402_1005Metric, F.Cu at (176.5, 63.8)
- added D2: BZX84Cxx, Package_TO_SOT_SMD:SOT-23, F.Cu at (152.1, 60.3)
- added D2: BZX84Cxx, Package_TO_SOT_SMD:SOT-23, F.Cu at (160.1, 60.2)
- added D2: BZX84Cxx, Package_TO_SOT_SMD:SOT-23, F.Cu at (136.9, 54.3)
- added D2: BZX84Cxx, Package_TO_SOT_SMD:SOT-23, F.Cu at (148.1, 60.2)
- added D2: BZX84Cxx, Package_TO_SOT_SMD:SOT-23, F.Cu at (172.5, 70.2)
- added D2: BZX84Cxx, Package_TO_SOT_SMD:SOT-23, F.Cu at (168.1, 60.3)
- added D2: BZX84Cxx, Package_TO_SOT_SMD:SOT-23, F.Cu at (164.1, 60.2)
- added D2: BZX84Cxx, Package_TO_SOT_SMD:SOT-23, F.Cu at (156.1, 60.2)
- added D20: LED, LED_SMD:LED_0402_1005Metric, F.Cu at (176.5, 62.2)
- added D21: LED, LED_SMD:LED_0402_1005Metric, F.Cu at (176.5, 60.8)
- added R90: 60R, Resistor_SMD:R_0402_1005Metric, F.Cu at (124.3, 79.4)
- added R91: 60R, Resistor_SMD:R_0402_1005Metric, F.Cu at (124.3, 77.4)
- added REF**: Harwin_LTek-Male_2x05_P2.00mm_Vertical, Connector_Harwin:Harwin_LTek-Male_2x05_P2.00mm_Vertical, F.Cu at (117.5, 79.4)
- added REF**: Molex_Micro-Fit_3.0_43045-0800_2x04_P3.00mm_Horizontal, SUFST:Molex_Micro-Fit_3.0_43045-0800_2x04_P3.00mm_Horizontal, F.Cu at (171.0, 45.0)
- added REF**: Harwin_LTek-Male_2x22_P2.00mm_Vertical, Connector_Harwin:Harwin_LTek-Male_2x22_P2.00mm_Vertical, F.Cu at (188.5, 53.8)
- added REF**: Harwin_LTek-Male_17_P2.00mm_Vertical, Connector_Harwin:Harwin_LTek-Male_17_P2.00mm_Vertical, F.Cu at (212.5, 100.5)
- added REF**: L_0805_2012Metric, Inductor_SMD:L_0805_2012Metric, F.Cu at (141.4, 64.5)
- added REF**: BUS_PCI_Express_Mini, Connector_PCBEdge:BUS_PCI_Express_Mini, F.Cu at (138.0, 89.0)
- added U14: LTC2875-DD, Package_DFN_QFN:DFN-8-1EP_3x3mm_P0.5mm_EP1.66x2.38mm, F.Cu at (127.1, 78.5)
- J3: moved to B.Cu
- moved D21 160.5 mm to (203.5, 53.8), turned to 90 degrees
- moved D20 158.5 mm to (202.0, 53.8), turned to 90 degrees
- moved D19 156.5 mm to (200.5, 53.8), turned to 90 degrees
- moved D18 154.5 mm to (199.0, 53.8), turned to 90 degrees
- moved R68 154.5 mm to (202.5, 59.9)
- moved R67 153.7 mm to (202.5, 60.9)
- moved R66 153.0 mm to (202.5, 61.9)
- moved D17 152.5 mm to (197.5, 53.8), turned to 90 degrees
- moved R65 152.4 mm to (202.5, 62.9)
- moved D16 150.5 mm to (196.0, 53.8), turned to 90 degrees
- moved R70 149.2 mm to (201.7, 57.1), turned to -90 degrees
- moved R75 148.8 mm to (198.7, 57.1), turned to -90 degrees
- moved R71 148.6 mm to (200.7, 57.1), turned to -90 degrees
- moved D15 148.6 mm to (194.5, 53.8), turned to 90 degrees
- moved R72 148.2 mm to (199.7, 57.1), turned to -90 degrees
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